File: Arrow PCB/DDR Pad.sch (KiCad schematic (older format))
At the start: 39 parts, among them J10 RJ45, J9 Conn_01x03

Commit message: Update Arrow schematic. Add schematic images.
Other:
- note added: "To Teensy Board"
- note removed: "To Teensy Board\nFootprint on four sides of board,\nonly one needs to be populated"
Changed lines of the file:
@@
 EESchema Schematic File Version 4
+LIBS:DDR Pad-cache
 EELAYER 30 0
 EELAYER END
@@
 $EndComp
 Text Notes 8600 2750 0    50   ~ 0
-To Teensy Board\nFootprint on four sides of board,\nonly one needs to be populated
+To Teensy Board
 $Comp
 L Connector_Generic:Conn_01x02 J_E_ZE1
